File: uMouse_prototype.sch (EAGLE design)
At the start: 76 parts, among them IC1 LM1117IMPX-5.0, IC2 LM1117IMPX-5.0

Commit message: gotowa, czeka na uwagi Tomka i Kuby
Parts:
- added C27: 100nF 6.3V, rcl:C-EUC0805K
- added U$2: (no value), Nordic_nRF:INDUCTOR_0805_L
Connections:
- removed net AGND: C18.2, C19.2, C20.2, C21.2, C22.2, PT1.C, PT2.C, PT3.C, PT4.C, PT5.C, R19.1, R22.1, U$5.AGND
- removed net N$25: U$5.PA15
- new net N$22: U$2.2, U$5.AVDD
- net 7.4V/VBAT: now also C25.1, C26.1, U$3.VBB
- net GND: now also C18.2, C19.2, C20.2, C21.2, C22.2, C27.2, PT1.C, PT2.C, PT3.C, PT4.C, PT5.C, R19.1, R22.1, U$5.AGND, U$5.GND_1, U$5.GND_2, U$5.GND_3, U$5.GND_4, U$5.GND_5
- net LEFT-ENC-A: now also JP2.3, U$5.PA0; no longer JP1.1, U$5.PC10
- net LEFT-ENC-B: now also JP2.1, U$5.PA1; no longer JP1.3, U$5.PC12
- net LEFT-M-OUT1: now also JP2.2, U$3.OUT1; no longer JP1.2, U$1.OUT1
- net LEFT-M-OUT2: now also JP2.4, U$3.OUT2; no longer JP1.4, U$1.OUT2
- net LEFT-M-PWM1: now also U$3.IN1, U$5.PC8; no longer U$1.IN1, U$5.PB10, U$5.PC6
- net LEFT-M-PWM2: now also U$3.IN2, U$5.PC6; no longer U$1.IN2, U$5.PC7
- net RECEIVER_1: now also U$5.PA6; no longer U$5.PA0
- net RECEIVER_2: now also U$5.PA5; no longer U$5.PA1
- net RIGHT-ENC-A: now also JP1.3, U$5.PA9; no longer JP2.1, U$5.PA13
- net RIGHT-ENC-B: now also JP1.1, U$5.PA8; no longer JP2.3, U$5.PA14
- net RIGHT-M-OUT1: now also JP1.2, U$1.OUT1; no longer JP2.2, U$3.OUT1
- net RIGHT-M-OUT2: now also JP1.4, U$1.OUT2; no longer JP2.4, U$3.OUT2
- net RIGHT-M-PWM1: now also U$1.IN1, U$5.PC9; no longer U$3.IN1, U$5.PB3, U$5.PC8
- net RIGHT-M-PWM2: now also U$1.IN2, U$5.PC7; no longer U$3.IN2, U$5.PB4, U$5.PC9
- net VBAT: no longer C25.1, C26.1, U$3.VBB
- net VCC: now also C27.1, U$2.1

Commit message: ostatnie poprawki, plytka do enkoderow
Parts:
- added C28: 1uF 16V, rcl:C-EUC0805K
- added C29: 4.7uF 6.3V, rcl:C-EUC0805K
- added C30: 100nF 6.3V, rcl:C-EUC0805K
- added IC3: LM1117IMPX-5.0, lm1117:LM1117IMPX-5.0
- added JP3, JP4: (no value), pinhead:PINHD-1X2
- added JP5: (no value), pinhead:PINHD-1X6
Connections:
- new net 5V: C29.1, C30.1, IC3.OUT, IC3.OUT1, JP5.5
- new net EN: JP5.6
- new net RX-STM: JP5.3, U$5.PC5
- new net STATE: JP5.1
- new net TX-STM: JP5.2, U$5.PB10
- net 7.4V/VBAT: now also C28.1, IC3.IN
- net GND: now also C28.2, C29.2, C30.2, IC3.GND, JP5.4
- net LEFT-M-OUT1: now also JP4.1
- net LEFT-M-OUT2: now also JP4.2
- net RIGHT-M-OUT1: now also JP3.1
- net RIGHT-M-OUT2: now also JP3.2
Other:
- note added: "LDO 7.4V->5V"
Changed lines of the file:
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@@
 <part name="GND41" library="supply1" library_urn="urn:adsk.eagle:library:371" deviceset="GND" device=""/>
 <part name="GND42" library="supply1" library_urn="urn:adsk.eagle:library:371" deviceset="GND" device=""/>
+<part name="JP3" library="pinhead" library_urn="urn:adsk.eagle:library:325" deviceset="PINHD-1X2" device="" package3d_urn="urn:adsk.eagle:package:22435/2"/>
+<part name="JP4" library="pinhead" library_urn="urn:adsk.eagle:library:325" deviceset="PINHD-1X2" device="" package3d_urn="urn:adsk.eagle:package:22435/2"/>
+<part name="IC3" library="lm1117" deviceset="LM1117IMPX-*" device="" technology="5.0"/>
+<part name="C28" library="rcl" library_urn="urn:adsk.eagle:library:334" deviceset="C-EU" device="C0805K" value="1uF 16V"/>
+<part name="GND43" library="supply1" library_urn="urn:adsk.eagle:library:371" deviceset="GND" device=""/>
+<part name="GND44" library="supply1" library_urn="urn:adsk.eagle:library:371" deviceset="GND" device=""/>
+<part name="C29" library="rcl" library_urn="urn:adsk.eagle:library:334" deviceset="C-EU" device="C0805K" value="4.7uF 6.3V"/>
+<part name="GND45" library="supply1" library_urn="urn:adsk.eagle:library:371" deviceset="GND" device=""/>
+<part name="C30" library="rcl" library_urn="urn:adsk.eagle:library:334" deviceset="C-EU" device="C0805K" value="100nF 6.3V"/>
+<part name="GND46" library="supply1" library_urn="urn:adsk.eagle:library:371" deviceset="GND" device=""/>
+<part name="JP5" library="pinhead" library_urn="urn:adsk.eagle:library:325" deviceset="PINHD-1X6" device="" package3d_urn="urn:adsk.eagle:package:22472/2"/>
 </parts>
 <sheets>
@@
 <text x="236.22" y="-271.78" size="5.08" layer="97">Right motor</text>
 <text x="-66.04" y="114.3" size="1.778" layer="97">LDO 7.4V-&gt;3.3V</text>
+<text x="-55.88" y="27.94" size="1.778" layer="97">LDO 7.4V-&gt;5V</text>
 </plain>
 <instances>
@@
 <instance part="GND41" gate="1" x="142.24" y="124.46"/>
 <instance part="GND42" gate="1" x="177.8" y="83.82"/>
+<instance part="JP3" gate="G$1" x="223.52" y="-139.7"/>
+<instance part="JP4" gate="G$1" x="226.06" y="-243.84" rot="MR180"/>
+<instance part="IC3" gate="G$1" x="-48.26" y="20.32"/>
+<instance part="C28" gate="G$1" x="-66.04" y="15.24"/>
+<instance part="GND43" gate="1" x="-66.04" y="2.54"/>
+<instance part="GND44" gate="1" x="-48.26" y="2.54"/>
+<instance part="C29" gate="G$1" x="-22.86" y="15.24"/>
+<instance part="GND45" gate="1" x="-22.86" y="2.54"/>
+<instance part="C30" gate="G$1" x="-5.08" y="15.24"/>
+<instance part="GND46" gate="1" x="-5.08" y="2.54"/>
+<instance part="JP5" gate="A" x="-35.56" y="-22.86"/>
 </instances>
 <busses>
@@
 <junction x="152.4" y="-223.52"/>
 </segment>
+<segment>
+<pinref part="IC3" gate="G$1" pin="IN"/>
+<wire x1="-55.88" y1="20.32" x2="-66.04" y2="20.32" width="0.1524" layer="91"/>
+<label x="-73.66" y="20.32" size="1.016" layer="95" rot="R180" xref="yes"/>
+<pinref part="C28" gate="G$1" pin="1"/>
+<wire x1="-66.04" y1="20.32" x2="-73.66" y2="20.32" width="0.1524" layer="91"/>
+<wire x1="-66.04" y1="17.78" x2="-66.04" y2="20.32" width="0.1524" layer="91"/>
+<junction x="-66.04" y="20.32"/>
+</segment>
 </net>
 <net name="GND" class="0">
@@
 <wire x1="177.8" y1="88.9" x2="177.8" y2="86.36" width="0.1524" layer="91"/>
 <pinref part="GND42" gate="1" pin="GND"/>
+</segment>
+<segment>
+<pinref part="C28" gate="G$1" pin="2"/>
+<wire x1="-66.04" y1="10.16" x2="-66.04" y2="5.08" width="0.1524" layer="91"/>
+<pinref part="GND43" gate="1" pin="GND"/>
+</segment>
+<segment>
+<pinref part="IC3" gate="G$1" pin="GND"/>
+<wire x1="-48.26" y1="12.7" x2="-48.26" y2="5.08" width="0.1524" layer="91"/>
+<pinref part="GND44" gate="1" pin="GND"/>
+</segment>
+<segment>
+<pinref part="C29" gate="G$1" pin="2"/>
+<wire x1="-22.86" y1="10.16" x2="-22.86" y2="5.08" width="0.1524" layer="91"/>
+<pinref part="GND45" gate="1" pin="GND"/>
+</segment>
+<segment>
+<pinref part="C30" gate="G$1" pin="2"/>
+<wire x1="-5.08" y1="10.16" x2="-5.08" y2="5.08" width="0.1524" layer="91"/>
+<pinref part="GND46" gate="1" pin="GND"/>
+</segment>
+<segment>
+<pinref part="JP5" gate="A" pin="4"/>
+<wire x1="-38.1" y1="-22.86" x2="-45.72" y2="-22.86" width="0.1524" layer="91"/>
+<label x="-45.72" y="-22.86" size="1.016" layer="95" rot="R180" xref="yes"/>
 </segment>
 </net>
@@
 <pinref part="JP1" gate="A" pin="2"/>
 </segment>
+<segment>
+<pinref part="JP3" gate="G$1" pin="1"/>
+<wire x1="220.98" y1="-137.16" x2="210.82" y2="-137.16" width="0.1524" layer="91"/>
+<label x="210.82" y="-137.16" size="1.016" layer="95" rot="R180" xref="yes"/>
+</segment>
 </net>
 <net name="RIGHT-M-OUT2" class="0">
@@
 <label x="231.14" y="-114.3" size="1.016" layer="95" xref="yes"/>
 <pinref part="JP1" gate="A" pin="4"/>
+</segment>
+<segment>
+<pinref part="JP3" gate="G$1" pin="2"/>
+<wire x1="220.98" y1="-139.7" x2="210.82" y2="-139.7" width="0.1524" layer="91"/>
+<label x="210.82" y="-139.7" size="1.016" layer="95" rot="R180" xref="yes"/>
 </segment>
 </net>
@@
 <pinref part="JP2" gate="A" pin="4"/>
 </segment>
+<segment>
+<pinref part="JP4" gate="G$1" pin="2"/>
+<wire x1="223.52" y1="-243.84" x2="213.36" y2="-243.84" width="0.1524" layer="91"/>
+<label x="213.36" y="-243.84" size="1.016" layer="95" rot="MR0" xref="yes"/>
+</segment>
 </net>
 <net name="LEFT-M-OUT1" class="0">
@@
 <label x="233.68" y="-213.36" size="1.016" layer="95" xref="yes"/>
 <pinref part="JP2" gate="A" pin="2"/>
+</segment>
+<segment>
+<pinref part="JP4" gate="G$1" pin="1"/>
+<wire x1="223.52" y1="-246.38" x2="213.36" y2="-246.38" width="0.1524" layer="91"/>
+<label x="213.36" y="-246.38" size="1.016" layer="95" rot="MR0" xref="yes"/>
 </segment>
 </net>
@@
 </segment>
 </net>
+<net name="5V" class="0">
+<segment>
+<pinref part="IC3" gate="G$1" pin="OUT"/>
+<wire x1="-40.64" y1="20.32" x2="-35.56" y2="20.32" width="0.1524" layer="91"/>
+<pinref part="IC3" gate="G$1" pin="OUT1"/>
+<wire x1="-40.64" y1="22.86" x2="-35.56" y2="22.86" width="0.1524" layer="91"/>
+<wire x1="-35.56" y1="22.86" x2="-35.56" y2="20.32" width="0.1524" layer="91"/>
+<junction x="-35.56" y="20.32"/>
+<wire x1="-35.56" y1="20.32" x2="-22.86" y2="20.32" width="0.1524" layer="91"/>
+<label x="5.08" y="20.32" size="1.016" layer="95" xref="yes"/>
+<pinref part="C29" gate="G$1" pin="1"/>
+<wire x1="-22.86" y1="20.32" x2="-5.08" y2="20.32" width="0.1524" layer="91"/>
+<wire x1="-5.08" y1="20.32" x2="5.08" y2="20.32" width="0.1524" layer="91"/>
+<wire x1="-22.86" y1="17.78" x2="-22.86" y2="20.32" width="0.1524" layer="91"/>
+<junction x="-22.86" y="20.32"/>
+<pinref part="C30" gate="G$1" pin="1"/>
+<wire x1="-5.08" y1="17.78" x2="-5.08" y2="20.32" width="0.1524" layer="91"/>
+<junction x="-5.08" y="20.32"/>
+</segment>
+<segment>
+<pinref part="JP5" gate="A" pin="5"/>
+<wire x1="-38.1" y1="-25.4" x2="-45.72" y2="-25.4" width="0.1524" layer="91"/>
+<label x="-45.72" y="-25.4" size="1.016" layer="95" rot="R180" xref="yes"/>
+</segment>
+</net>
+<net name="STATE" class="0">
+<segment>
+<pinref part="JP5" gate="A" pin="1"/>
+<wire x1="-38.1" y1="-15.24" x2="-45.72" y2="-15.24" width="0.1524" layer="91"/>
+<label x="-45.72" y="-15.24" size="1.016" layer="95" rot="R180" xref="yes"/>
+</segment>
+</net>
+<net name="TX-STM" class="0">
+<segment>
+<pinref part="JP5" gate="A" pin="2"/>
+<wire x1="-38.1" y1="-17.78" x2="-45.72" y2="-17.78" width="0.1524" layer="91"/>
+<label x="-45.72" y="-17.78" size="1.016" layer="95" rot="R180" xref="yes"/>
+</segment>
+<segment>
+<pinref part="U$5" gate="G$1" pin="PB10"/>
+<wire x1="134.62" y1="81.28" x2="132.08" y2="81.28" width="0.1524" layer="91"/>
+<wire x1="132.08" y1="81.28" x2="132.08" y2="78.74" width="0.1524" layer="91"/>
+<wire x1="132.08" y1="78.74" x2="129.54" y2="78.74" width="0.1524" layer="91"/>
+<label x="129.54" y="78.74" size="1.016" layer="95" rot="R180" xref="yes"/>
+</segment>
+</net>
+<net name="RX-STM" class="0">
+<segment>
+<pinref part="JP5" gate="A" pin="3"/>
+<wire x1="-38.1" y1="-20.32" x2="-45.72" y2="-20.32" width="0.1524" layer="91"/>
+<label x="-45.72" y="-20.32" size="1.016" layer="95" rot="R180" xref="yes"/>
+</segment>
+<segment>
+<pinref part="U$5" gate="G$1" pin="PC5"/>
+<wire x1="170.18" y1="106.68" x2="175.26" y2="106.68" width="0.1524" layer="91"/>
+<label x="175.26" y="106.68" size="1.016" layer="95" xref="yes"/>
+</segment>
+</net>
+<net name="EN" class="0">
+<segment>
+<pinref part="JP5" gate="A" pin="6"/>
+<wire x1="-38.1" y1="-27.94" x2="-45.72" y2="-27.94" width="0.1524" layer="91"/>
+<label x="-45.72" y="-27.94" size="1.016" layer="95" rot="R180" xref="yes"/>
+</segment>
+</net>

Commit message: poprawione i2c, dodane otwory pod holderki do ledów IR (tylko przy dwóch)
Parts:
- added R25: 0R, rcl:R-EU_M0805
Connections:
- new net N$28: R25.2, U$5.VIN
- net 7.4V/VBAT: now also R25.1; no longer U$5.VIN
- net IR4_SIGNAL: now also U$5.PA13; no longer U$5.PF7
- net SCL: now also R24.2, U$5.PB7; no longer R24.1, U$5.PC0
- net SDA: now also R23.2, U$5.PB6; no longer R23.1, U$5.PC1
- net VCC: now also R23.1, R24.1; no longer R23.2, R24.2
Other:
- moved on the sheet: R23, R24
Changed lines of the file:
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@@
 <part name="PT5" library="adafruit" library_urn="urn:adsk.eagle:library:420" deviceset="LED" device="3MM"/>
 <part name="MPU-RESZTA-ŚWIATA" library="pinhead" library_urn="urn:adsk.eagle:library:325" deviceset="PINHD-1X8" device="" package3d_urn="urn:adsk.eagle:package:22409/2"/>
-<part name="R23" library="rcl" library_urn="urn:adsk.eagle:library:334" deviceset="R-EU_" device="M0805" value="1k"/>
-<part name="R24" library="rcl" library_urn="urn:adsk.eagle:library:334" deviceset="R-EU_" device="M0805" value="1k"/>
-<part name="SUPPLY2" library="supply2" library_urn="urn:adsk.eagle:library:372" deviceset="VCC" device=""/>
-<part name="SUPPLY28" library="supply2" library_urn="urn:adsk.eagle:library:372" deviceset="VCC" device=""/>
 <part name="SUPPLY29" library="supply2" library_urn="urn:adsk.eagle:library:372" deviceset="VCC" device=""/>
 <part name="SUPPLY30" library="supply2" library_urn="urn:adsk.eagle:library:372" deviceset="VCC" device=""/>
@@
 <part name="GND46" library="supply1" library_urn="urn:adsk.eagle:library:371" deviceset="GND" device=""/>
 <part name="JP5" library="pinhead" library_urn="urn:adsk.eagle:library:325" deviceset="PINHD-1X6" device="" package3d_urn="urn:adsk.eagle:package:22472/2"/>
+<part name="R25" library="rcl" library_urn="urn:adsk.eagle:library:334" deviceset="R-EU_" device="M0805" value="0R"/>
+<part name="R23" library="rcl" library_urn="urn:adsk.eagle:library:334" deviceset="R-EU_" device="M0805" value="1k"/>
+<part name="R24" library="rcl" library_urn="urn:adsk.eagle:library:334" deviceset="R-EU_" device="M0805" value="1k"/>
+<part name="SUPPLY2" library="supply2" library_urn="urn:adsk.eagle:library:372" deviceset="VCC" device=""/>
+<part name="SUPPLY28" library="supply2" library_urn="urn:adsk.eagle:library:372" deviceset="VCC" device=""/>
 </parts>
 <sheets>
@@
 <instance part="PT5" gate="G$1" x="614.68" y="15.24"/>
 <instance part="MPU-RESZTA-ŚWIATA" gate="A" x="226.06" y="40.64"/>
-<instance part="R23" gate="G$1" x="111.76" y="45.72" rot="R270"/>
-<instance part="R24" gate="G$1" x="119.38" y="45.72" rot="R270"/>
-<instance part="SUPPLY2" gate="G$1" x="129.54" y="40.64"/>
-<instance part="SUPPLY28" gate="G$1" x="104.14" y="40.64"/>
 <instance part="SUPPLY29" gate="G$1" x="-12.7" y="149.86"/>
 <instance part="SUPPLY30" gate="G$1" x="-12.7" y="111.76" rot="MR0"/>
@@
 <instance part="GND46" gate="1" x="-5.08" y="2.54"/>
 <instance part="JP5" gate="A" x="-35.56" y="-22.86"/>
+<instance part="R25" gate="G$1" x="116.84" y="53.34" rot="R180"/>
+<instance part="R23" gate="G$1" x="205.74" y="53.34" rot="R270"/>
+<instance part="R24" gate="G$1" x="198.12" y="53.34" rot="R270"/>
+<instance part="SUPPLY2" gate="G$1" x="198.12" y="63.5"/>
+<instance part="SUPPLY28" gate="G$1" x="205.74" y="63.5"/>
 </instances>
 <busses>
@@
 </segment>
 <segment>
-<pinref part="U$5" gate="G$1" pin="VIN"/>
-<wire x1="109.22" y1="83.82" x2="121.92" y2="81.28" width="0.1524" layer="91"/>
-<label x="121.92" y="81.28" size="1.016" layer="95" xref="yes"/>
+<label x="124.46" y="53.34" size="1.016" layer="95" xref="yes"/>
+<pinref part="R25" gate="G$1" pin="1"/>
+<wire x1="121.92" y1="53.34" x2="124.46" y2="53.34" width="0.1524" layer="91"/>
 </segment>
 <segment>
@@
 </segment>
 <segment>
-<pinref part="R24" gate="G$1" pin="2"/>
-<wire x1="119.38" y1="40.64" x2="119.38" y2="35.56" width="0.1524" layer="91"/>
-<wire x1="119.38" y1="35.56" x2="129.54" y2="35.56" width="0.1524" layer="91"/>
-<wire x1="129.54" y1="35.56" x2="129.54" y2="38.1" width="0.1524" layer="91"/>
-<pinref part="SUPPLY2" gate="G$1" pin="VCC"/>
-</segment>
-<segment>
-<pinref part="R23" gate="G$1" pin="2"/>
-<wire x1="111.76" y1="40.64" x2="111.76" y2="35.56" width="0.1524" layer="91"/>
-<wire x1="111.76" y1="35.56" x2="104.14" y2="35.56" width="0.1524" layer="91"/>
-<wire x1="104.14" y1="35.56" x2="104.14" y2="38.1" width="0.1524" layer="91"/>
-<pinref part="SUPPLY28" gate="G$1" pin="VCC"/>
-</segment>
-<segment>
 <pinref part="C7" gate="G$1" pin="1"/>
 <pinref part="SUPPLY30" gate="G$1" pin="VCC"/>
@@
 <junction x="127" y="142.24"/>
 </segment>
+<segment>
+<pinref part="R24" gate="G$1" pin="1"/>
+<wire x1="198.12" y1="58.42" x2="198.12" y2="60.96" width="0.1524" layer="91"/>
+<pinref part="SUPPLY2" gate="G$1" pin="VCC"/>
+</segment>
+<segment>
+<pinref part="R23" gate="G$1" pin="1"/>
+<wire x1="205.74" y1="58.42" x2="205.74" y2="60.96" width="0.1524" layer="91"/>
+<pinref part="SUPPLY28" gate="G$1" pin="VCC"/>
+</segment>
 </net>
 <net name="N$5" class="0">
@@
 </segment>
 <segment>
-<pinref part="U$5" gate="G$1" pin="PF7"/>
-<wire x1="73.66" y1="99.06" x2="68.58" y2="99.06" width="0.1524" layer="91"/>
-<label x="68.58" y="99.06" size="1.27" layer="95" rot="R180" xref="yes"/>
+<label x="68.58" y="96.52" size="1.27" layer="95" rot="R180" xref="yes"/>
+<pinref part="U$5" gate="G$1" pin="PA13"/>
+<wire x1="73.66" y1="96.52" x2="68.58" y2="96.52" width="0.1524" layer="91"/>
 </segment>
 </net>
@@
 <net name="SCL" class="0">
 <segment>
-<pinref part="U$5" gate="G$1" pin="PC0"/>
-<wire x1="109.22" y1="66.04" x2="109.22" y2="58.42" width="0.1524" layer="91"/>
-<wire x1="109.22" y1="58.42" x2="119.38" y2="58.42" width="0.1524" layer="91"/>
-<label x="121.92" y="58.42" size="1.27" layer="95" xref="yes"/>
-<pinref part="R24" gate="G$1" pin="1"/>
-<wire x1="119.38" y1="58.42" x2="121.92" y2="58.42" width="0.1524" layer="91"/>
-<wire x1="119.38" y1="50.8" x2="119.38" y2="58.42" width="0.1524" layer="91"/>
-<junction x="119.38" y="58.42"/>
-</segment>
-<segment>
-<wire x1="223.52" y1="45.72" x2="215.9" y2="45.72" width="0.1524" layer="91"/>
-<label x="215.9" y="45.72" size="1.27" layer="95" rot="R180" xref="yes"/>
+<wire x1="223.52" y1="45.72" x2="198.12" y2="45.72" width="0.1524" layer="91"/>
+<label x="193.04" y="45.72" size="1.27" layer="95" rot="R180" xref="yes"/>
 <pinref part="MPU-RESZTA-ŚWIATA" gate="A" pin="3"/>
+<pinref part="R24" gate="G$1" pin="2"/>
+<wire x1="198.12" y1="45.72" x2="193.04" y2="45.72" width="0.1524" layer="91"/>
+<wire x1="198.12" y1="48.26" x2="198.12" y2="45.72" width="0.1524" layer="91"/>
+<junction x="198.12" y="45.72"/>
 </segment>
 <segment>
@@
 <label x="215.9" y="68.58" size="1.27" layer="95" rot="R180" xref="yes"/>
 </segment>
+<segment>
+<pinref part="U$5" gate="G$1" pin="PB7"/>
+<wire x1="73.66" y1="86.36" x2="68.58" y2="86.36" width="0.1524" layer="91"/>
+<label x="68.58" y="86.36" size="1.016" layer="95" rot="R180" xref="yes"/>
+</segment>
 </net>
 <net name="SDA" class="0">
 <segment>
-<pinref part="U$5" gate="G$1" pin="PC1"/>
-<wire x1="109.22" y1="68.58" x2="111.76" y2="68.58" width="0.1524" layer="91"/>
-<wire x1="111.76" y1="68.58" x2="111.76" y2="60.96" width="0.1524" layer="91"/>
-<wire x1="111.76" y1="60.96" x2="114.3" y2="60.96" width="0.1524" layer="91"/>
-<label x="114.3" y="60.96" size="1.27" layer="95" xref="yes"/>
-<pinref part="R23" gate="G$1" pin="1"/>
-<wire x1="111.76" y1="50.8" x2="111.76" y2="60.96" width="0.1524" layer="91"/>
-<junction x="111.76" y="60.96"/>
-</segment>
-<segment>
-<wire x1="223.52" y1="43.18" x2="215.9" y2="43.18" width="0.1524" layer="91"/>
-<label x="215.9" y="43.18" size="1.27" layer="95" rot="R180" xref="yes"/>
+<wire x1="223.52" y1="43.18" x2="205.74" y2="43.18" width="0.1524" layer="91"/>
+<label x="193.04" y="43.18" size="1.27" layer="95" rot="R180" xref="yes"/>
 <pinref part="MPU-RESZTA-ŚWIATA" gate="A" pin="4"/>
+<pinref part="R23" gate="G$1" pin="2"/>
+<wire x1="205.74" y1="43.18" x2="193.04" y2="43.18" width="0.1524" layer="91"/>
+<wire x1="205.74" y1="48.26" x2="205.74" y2="43.18" width="0.1524" layer="91"/>
+<junction x="205.74" y="43.18"/>
 </segment>
 <segment>
@@
 <wire x1="223.52" y1="71.12" x2="215.9" y2="71.12" width="0.1524" layer="91"/>
 <label x="215.9" y="71.12" size="1.27" layer="95" rot="R180" xref="yes"/>
+</segment>
+<segment>
+<pinref part="U$5" gate="G$1" pin="PB6"/>
+<wire x1="134.62" y1="91.44" x2="129.54" y2="91.44" width="0.1524" layer="91"/>
+<label x="129.54" y="91.44" size="1.016" layer="95" rot="R180" xref="yes"/>
 </segment>
 </net>
@@
 </segment>
 </net>
+<net name="N$28" class="0">
+<segment>
+<pinref part="U$5" gate="G$1" pin="VIN"/>
+<wire x1="109.22" y1="83.82" x2="111.76" y2="83.82" width="0.1524" layer="91"/>
+<wire x1="111.76" y1="83.82" x2="111.76" y2="53.34" width="0.1524" layer="91"/>
+<pinref part="R25" gate="G$1" pin="2"/>
+</segment>
+</net>
