File: uMouse_prototype/uMouse_prototype.brd (EAGLE design)
At the start: 90 x 100 mm, 86 parts, among them IC1 LM1117IMPX-5.0, IC2 LM1117IMPX-5.0, IC3 LM1117IMPX-5.0

Commit message: dodane gerbery do glownej plyty prototypu
Parts:
- renumbered MPU-RESZTA-ŚWIATA to MPU-RESZTA-SWIATA
Routing:
- net VCC: track 325.7 -> 331.9 mm
